File: NoisyCricket.sch (KiCad schematic (older format))
At the start: 9 parts, among them J1 +9 V, J2 Audio-Jack-2_Switch, Q1 J201

Commit message: complete with elements
Parts:
- added C1, C8: 220mF, Capacitors_THT:CP_Radial_D18.0mm_P7.50mm, symbol CP
- added C3: 100mF, Capacitors_THT:CP_Radial_D13.0mm_P7.50mm, symbol CP
- added C4, C5, C6: 100n, Capacitors_THT:C_Disc_D7.5mm_W5.0mm_P10.00mm, symbol C
- added C7: 47n, Capacitors_THT:C_Disc_D7.5mm_W5.0mm_P10.00mm, symbol C
- added J3: +9 V, Pin_Headers:Pin_Header_Straight_1x02_Pitch2.00mm, symbol Conn_01x01
- added J4: Headphones plug, Pin_Headers:Pin_Header_Straight_1x03_Pitch2.00mm, symbol Audio-Jack-2_Switch
- added LS1: Speaker, Pin_Headers:Pin_Header_Straight_1x02_Pitch2.00mm, symbol Speaker
- added R4, R5: 10, Resistors_THT:R_Axial_DIN0614_L14.3mm_D5.7mm_P7.62mm_Vertical, symbol R
- added SW1: SW_DIP_x01, Buttons_Switches_THT:SW_DIP_x1_W7.62mm_Slide_LowProfile, symbol SW_DIP_x01
- added U1: LM386, Housings_DIP:DIP-8_W7.62mm, symbol LM386
- added VR2: 1K, Potentiometers:Potentiometer_Alps_RK09Y_Vertical, symbol POT
- added VR3: 100K, Potentiometers:Potentiometer_Alps_RK09Y_Vertical, symbol POT
- C2: renamed from C1; value C -> 47n
- R1: value R -> 1M
- R2: value R -> 3K3
- R3: value R -> 4k7
- VR1: renamed from RV1; value POT -> 10K
Connections:
- net GND: now also C1.2, C3.2, C5.1, C7.1, LS1.2, R5.2, U1.3 (+), U1.4 (Gnd); no longer D1.1 (K)
- net at VR1.2: now also C6.2, VR3.1
- new net: C5.2, VR3.2, VR3.3
- new net: U1.1, VR2.1
- new net: C6.1, U1.2 (-)
- new net: C8.1, U1.5
- new net: C1.1, J3.1 (Pin_1), U1.6 (V+)
- new net: C3.1, U1.7
- new net: U1.8, VR2.2, VR2.3
- new net: C8.2, J4.1, J4.2, R5.1
- new net: C4.2, SW1.2
- new net: C7.2, R4.2
- new net: J4.3, LS1.1
Other:
- moved on the sheet: D1, J1, R3

Commit message: good for now
Parts:
- removed J1, J3: +9 V, Pin_Headers:Pin_Header_Straight_1x02_Pitch2.00mm, symbol Conn_01x01
- removed VR1: 10K, Potentiometers:Potentiometer_Alps_RK09Y_Vertical, symbol POT
- removed VR2: 1K, Potentiometers:Potentiometer_Alps_RK09Y_Vertical, symbol POT
- removed VR3: 100K, Potentiometers:Potentiometer_Alps_RK09Y_Vertical, symbol POT
- added BT1: Battery_Cell, Pin_Headers:Pin_Header_Straight_1x02_Pitch2.54mm, symbol Battery_Cell
- added GAIN1, INPUT1, TONE1: 10k, DARKO:Pin_Header_Straight_1x03_Pitch2.54mm, symbol POT-NOISY
- C1, C8: footprint Capacitors_THT:CP_Radial_D18.0mm_P7.50mm -> Capacitors_THT:CP_Radial_D12.5mm_P2.50mm
- J4: value Headphones plug -> Headphones
- R1, R2, R3, R4, R5: footprint Resistors_THT:R_Axial_DIN0614_L14.3mm_D5.7mm_P7.62mm_Vertical -> Resistors_THT:R_Axial_DIN0411_L9.9mm_D3.6mm_P7.62mm_Vertical
- input1: renamed from J2; value Audio-Jack-2_Switch -> audio input
Connections:
- net GND: now also D1.1 (K), BT1.2 (-), INPUT1.3
- net at Q1.1 (D), R3.2: now also C1.1, U1.6 (V+), BT1.1 (+)
- net at C2.1: now also INPUT1.1
- net at C6.2: now also INPUT1.2, TONE1.1
- net at C5.2: now also TONE1.2, TONE1.3
- net at U1.1: now also GAIN1.1
- net at C8.1, U1.5: now also C4.1, R4.1
- net at C3.1, U1.7: now also SW1.1
- net at U1.8: now also GAIN1.2, GAIN1.3
Other:
- moved on the sheet: C1, C2, C3, C4, C5, C6, C7, C8, D1, J4, LS1, Q1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
